File: Netzteil_CA1.brd (EAGLE design)
At the start: 56 x 77.5 mm, 83 parts, among them IC1 LM317T, IC2 MAX4080T, IC3 LM324, IC4 7805TV, IC5 LM334, IC7 MCP1541, IC8 MCP4922, IC9 LM358, Q1 16MHz, T1 TIP3055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

Commit message: move a via
Routing:
- net AGND: track 65.4 -> 66.0 mm
Changed lines of the file:
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@@
 </element>
 <element name="C34" library="goujine" package="0805" value="100n/16V" x="23.97125" y="48.3790625" smashed="yes">
-<attribute name="NAME" x="23.1775" y="49.3316125" size="0.8128" layer="25"/>
+<attribute name="NAME" x="23.5346375" y="49.37125" size="0.8128" layer="25" rot="R90"/>
 <attribute name="OC_MOUSER" value="810-C2012X7R2A104K" x="23.97125" y="48.3790625" size="1.778" layer="27" display="off"/>
 <attribute name="VALUE" x="26.19375" y="47.2677625" size="1.016" layer="27"/>
@@
 </element>
 <element name="BTN" library="neumluc" package="JST-PH-2.0-4P" value="" x="28.8925" y="53.49875" smashed="yes" rot="R90">
-<attribute name="NAME" x="26.67" y="46.25975" size="0.8128" layer="25" ratio="10"/>
+<attribute name="NAME" x="26.67" y="46.4185" size="0.8128" layer="25" ratio="10"/>
 <attribute name="OC_DIGIKEY" value="455-1706-ND" x="28.8925" y="53.49875" size="1.778" layer="27" rot="R90" display="off"/>
 <attribute name="VALUE" x="33.87725" y="47.14875" size="0.8128" layer="27" ratio="10" rot="R90"/>
@@
 <wire x1="19.52625" y1="50.165" x2="19.7246875" y2="49.9665625" width="0.4064" layer="1"/>
 <wire x1="19.7246875" y1="49.9665625" x2="21.19875" y2="49.9665625" width="0.4064" layer="1"/>
-<via x="24.28875" y="46.83125" extent="1-16" drill="0.35"/>
-<wire x1="24.28875" y1="46.83125" x2="25.4" y2="46.83125" width="0.8128" layer="1"/>
 <wire x1="25.4" y1="46.83125" x2="26.035" y2="46.83125" width="0.8128" layer="1"/>
 <wire x1="26.035" y1="46.83125" x2="25.6778125" y2="46.7121875" width="0.8128" layer="1"/>
@@
 <contactref element="PANEL" pad="1"/>
 <contactref element="SERIAL" pad="3"/>
+<via x="24.28875" y="49.8475" extent="1-16" drill="0.35"/>
+<wire x1="24.28875" y1="49.8475" x2="24.92375" y2="49.2125" width="0.8128" layer="1"/>
+<wire x1="24.92375" y1="49.2125" x2="24.92375" y2="48.3790625" width="0.8128" layer="1"/>
 </signal>
 <signal name="N$5">
